Commit message: added full field configuration

File: rocket_league_simulation/util/urdf/backwall.urdf (robot description, URDF)
Before this commit: robot goal, 1 links, 0 joints
Links:
- link base_link: geometry collision box size=10. 0.25 0.25; visual box size=10. 0.25 0.25

File: rocket_league_simulation/util/urdf/car.urdf (robot description, URDF)
Before this commit: robot simplecar, 1 links, 0 joints
Links:
- link base_link: geometry collision box size=.3 0.15 0.1; visual box size=0.3 0.15 0.1

File: rocket_league_simulation/util/urdf/sidewall.urdf (robot description, URDF)
Before this commit: robot goal, 1 links, 0 joints
Links:
- link base_link: geometry collision box size=0.25 15. 0.25; visual box size=0.25 15. 0.25
