Commit message: fixed minor errorsg

File: rocket_league_simulation/urdf/backwall.urdf (robot description, URDF)
Before this commit: robot backwall, 1 links, 0 joints
Links:
- link base_link: geometry collision box size=1.067 0.25 0.25; visual box size=1.067 0.25 0.25

File: rocket_league_simulation/urdf/goal.urdf (robot description, URDF)
Before this commit: robot goal, 1 links, 0 joints
Links:
- link base_link: geometry collision box size=0.91435 0.25 0.25; visual box size=0.91435 0.25 0.25

File: rocket_league_simulation/urdf/sidewall.urdf (robot description, URDF)
Before this commit: robot sidewall, 1 links, 0 joints
Links:
- link base_link: geometry collision box size=0.25 4.572 0.25; visual box size=0.25 4.572 0.25

Commit message: centered and x-positive aligned

File: rocket_league_simulation/urdf/backwall.urdf (robot description, URDF)
Before this commit: robot backwall, 1 links, 0 joints
Links:
- link base_link: geometry collision box size=0.25 1.067 0.25; visual box size=0.25 1.067 0.25

File: rocket_league_simulation/urdf/car.urdf (robot description, URDF)
Before this commit: robot simplecar, 1 links, 0 joints
Links:
- link base_link: geometry collision box size=.13 0.28 0.1; visual box size=0.13 0.28 0.1

File: rocket_league_simulation/urdf/goal.urdf (robot description, URDF)
Before this commit: robot goal, 1 links, 0 joints
Links:
- link base_link: geometry collision box size=0.25 0.91435 0.25; visual box size=0.25 0.91435 0.25

File: rocket_league_simulation/urdf/sidewall.urdf (robot description, URDF)
Before this commit: robot sidewall, 1 links, 0 joints
Links:
- link base_link: geometry collision box size=4.572 0.25 0.25; visual box size=4.572 0.25 0.25
