Commit message: modified field size

File: rktl_sim/urdf/backwall.urdf (robot description, URDF)
Before this commit: robot backwall, 1 links, 0 joints
Links:
- link base_link: geometry collision box size=0.25 1.25 0.25; visual box size=0.25 1.25 0.25

File: rktl_sim/urdf/goal.urdf (robot description, URDF)
Before this commit: robot goal, 1 links, 0 joints
Links:
- link base_link: geometry collision box size=0.25 1.0 0.25; visual box size=0.25 1.0 0.25

File: rktl_sim/urdf/sidewall.urdf (robot description, URDF)
Before this commit: robot sidewall, 1 links, 0 joints
Links:
- link base_link: geometry collision box size=5.0 0.25 0.25; visual box size=5.0 0.25 0.25

Commit message: added restitution to field objects

File: rktl_sim/urdf/backwall.urdf (robot description, URDF)
Before this commit: robot backwall, 1 links, 0 joints
Links:
- link base_link: mass None -> 1.0

File: rktl_sim/urdf/ball.urdf (robot description, URDF)
Before this commit: robot simple_ball, 1 links, 0 joints
Links:
- removed link ball
- added link base_link, mass 0.1; collision sphere radius=0.05; visual sphere radius=0.05

File: rktl_sim/urdf/goal.urdf (robot description, URDF)
Before this commit: robot goal, 1 links, 0 joints
Links:
- link base_link: mass None -> 1.0

File: rktl_sim/urdf/plane.urdf (robot description, URDF)
Before this commit: robot plane, 1 links, 0 joints
Links:
- removed link planeLink
- added link base_link, mass 1.0; collision box size=200 200 10; visual mesh filename=plane100.obj scale=1 1 1

File: rktl_sim/urdf/sidewall.urdf (robot description, URDF)
Before this commit: robot sidewall, 1 links, 0 joints
Links:
- link base_link: mass None -> 1.0

Commit message: continued tuning

File: rktl_sim/urdf/backwall.urdf (robot description, URDF)
Before this commit: robot backwall, 1 links, 0 joints
Links:
- link base_link: mass 1.0 -> 100.0

File: rktl_sim/urdf/ball.urdf (robot description, URDF)
Before this commit: robot simple_ball, 1 links, 0 joints
Links:
- link base_link: mass 0.1 -> 0.001

File: rktl_sim/urdf/goal.urdf (robot description, URDF)
Before this commit: robot goal, 1 links, 0 joints
Links:
- link base_link: mass 1.0 -> 100.0

File: rktl_sim/urdf/sidewall.urdf (robot description, URDF)
Before this commit: robot sidewall, 1 links, 0 joints
Links:
- link base_link: mass 1.0 -> 100.0
