Commit message: added basic changes for initial speed on ball

File: rktl_sim/urdf/ball.urdf (robot description, URDF)
Before this commit: robot simple_ball, 1 links, 0 joints
Links:
- link ball: mass 1.0 -> 0.25; geometry collision sphere radius=0.05; visual mesh filename=ball.obj scale=1 1 1

Commit message: tuned ball physics slightly

File: rktl_sim/urdf/ball.urdf (robot description, URDF)
Before this commit: robot simple_ball, 1 links, 0 joints
Links:
- link base_link: mass 0.001 -> 10.
