Commit message: moved to joint model

File: rktl_sim/urdf/car.urdf (robot description, URDF)
Before this commit: robot simplecar, 1 links, 0 joints
Links:
- added link chassis, mass .1; collision box size=0.13 0.28 0.1; visual box size=0.13 0.28 0.1
- link base_link: geometry 
Joints:
- added joint base_link_joint: type prismatic, parent base_link, child chassis, origin xyz=0 0 0.5 rpy=0 0 0, axis 1 0 0, limit effort=100 velocity=10

Commit message: removed joint model

File: rktl_sim/urdf/car.urdf (robot description, URDF)
Before this commit: robot simplecar, 2 links, 1 joints
Links:
- removed link chassis
- link base_link: geometry collision box size=0.13 0.28 0.1; visual box size=0.13 0.28 0.1
Joints:
- removed joint base_link_joint

Commit message: fixed with joints

File: rktl_sim/urdf/car.urdf (robot description, URDF)
Before this commit: robot simplecar, 1 links, 0 joints
Links:
- added link car_link, mass 6; collision box size=0.13 0.28 0.1; visual box size=0.13 0.28 0.1
- added link w_link, mass 0
- added link x_link, mass 0
- link base_link: mass 6 -> 0; geometry 
Joints:
- added joint w_joint: type continuous, parent w_link, child car_link, origin xyz=0 0 0 rpy=0 0 0, axis 0 0 1
- added joint x_joint: type prismatic, parent x_link, child w_link, origin xyz=0 0 0 rpy=0 0 0, axis 0 1 0, limit lower=-100.0 upper=100.0 effort=500 velocity=500.0
- added joint y_joint: type prismatic, parent base_link, child x_link, origin xyz=0 0 0 rpy=0 0 0, axis 1 0 0, limit lower=-100.0 upper=100.0 effort=500 velocity=500.0

Commit message: wip; fixing framing

File: rktl_sim/urdf/car.urdf (robot description, URDF)
Before this commit: robot simplecar, 4 links, 3 joints
Joints:
- joint x_joint: axis 0 1 0 -> 1 0 0
- joint y_joint: axis 1 0 0 -> 0 1 0

Commit message: fixed frame issues

File: rktl_sim/urdf/car.urdf (robot description, URDF)
Before this commit: robot simplecar, 4 links, 3 joints
Links:
- link car_link: geometry collision box size=0.28 0.13 0.1; visual box size=0.28 0.13 0.1
