Commit message: fixed goal urdfs

File: rktl_sim/urdf/goal.urdf.xacro (robot description, xacro)
@@ -12,15 +12,15 @@
             <visual>
                 <geometry>
-                    <box size="${goal_size} 0.05 0.25"/>
+                    <box size="0.05 ${goal_size} 0.25"/>
                 </geometry>
             </visual>
             <collision>
                 <geometry>
-                    <box size="${goal_size} 0.05 0.25"/>
+                    <box size="0.05 ${goal_size} 0.25"/>
                 </geometry>
             </collision>
         </link>
         <joint name="goal_joint" type="fixed">
-            <origin xyz="0 ${x_dir*((field_length/2)+0.225)} 0" rpy="0 0 0" />
+            <origin xyz="${x_dir*((field_length/2)+0.175)} 0 0" rpy="0 0 0" />
             <parent link="base_link" />
             <child link="goal_link" />

File: rktl_sim/urdf/goal_a.urdf (robot description, URDF)
Before this commit: robot goal_a, 2 links, 1 joints
Joints:
- joint goal_joint: origin xyz=-2.3 0 0 rpy=0 0 0 -> xyz=2.3 0 0 rpy=0 0 0
